File: xmas-tree.kicad_sch (KiCad schematic)
At the start: 26 parts, among them U1 SN74HCS594, U2 LM555xM, U3 74AHC1G32

Commit message: Initial Commit
Parts:
- C1: value 0.1uf -> 0.01uf; footprint Capacitor_SMD:C_1210_3225Metric_Pad1.33x2.70mm_HandSolder -> Capacitor_SMD:C_0805_2012Metric_Pad1.18x1.45mm_HandSolder
- C2, C3: footprint Capacitor_SMD:C_1210_3225Metric_Pad1.33x2.70mm_HandSolder -> Capacitor_SMD:C_0805_2012Metric_Pad1.18x1.45mm_HandSolder
- R1, R2, R3, R4, R5, R6, R7, R8: footprint Resistor_SMD:R_2010_5025Metric -> Resistor_SMD:R_0805_2012Metric_Pad1.20x1.40mm_HandSolder
- R10: footprint Resistor_SMD:R_2010_5025Metric_Pad1.40x2.65mm_HandSolder -> Resistor_SMD:R_0805_2012Metric_Pad1.20x1.40mm_HandSolder
- R9: value 0 -> 2k; footprint Resistor_SMD:R_2010_5025Metric_Pad1.40x2.65mm_HandSolder -> Resistor_SMD:R_0805_2012Metric_Pad1.20x1.40mm_HandSolder
Other:
- note added: "This resistor has to be greater than 0 to not short circuit the thing"
Changed lines of the file:
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@@
     (effects (font (size 1.27 1.27)) (justify left bottom))
   )
+  (text "This resistor has to be greater than 0 to not short circuit the thing\n"
+    (at 202.565 41.275 0)
+    (effects (font (size 1.27 1.27)) (justify left bottom))
+  )
   (global_label "LED_H" (shape input) (at 87.63 55.88 270) (fields_autoplaced)
     (effects (font (size 1.27 1.27)) (justify right))
@@
       (effects (font (size 1.27 1.27)) (justify left))
     )
-    (property "Footprint" "Resistor_SMD:R_2010_5025Metric" (id 2) (at 72.771 43.434 90)
+    (property "Footprint" "Resistor_SMD:R_0805_2012Metric_Pad1.20x1.40mm_HandSolder" (id 2) (at 72.771 43.434 90)
       (effects (font (size 1.27 1.27)) hide)
     )
@@
       (effects (font (size 1.27 1.27)) (justify left))
     )
-    (property "Footprint" "Resistor_SMD:R_2010_5025Metric" (id 2) (at 41.021 43.434 90)
+    (property "Footprint" "Resistor_SMD:R_0805_2012Metric_Pad1.20x1.40mm_HandSolder" (id 2) (at 41.021 43.434 90)
       (effects (font (size 1.27 1.27)) hide)
     )
@@
     (in_bom yes) (on_board yes) (fields_autoplaced)
     (property "Reference" "C1" (id 0) (at 148.5836 47.1764 90))
-    (property "Value" "0.1uf" (id 1) (at 148.5836 49.9515 90))
-    (property "Footprint" "Capacitor_SMD:C_1210_3225Metric_Pad1.33x2.70mm_HandSolder" (id 2) (at 148.59 52.705 0)
+    (property "Value" "0.01uf" (id 1) (at 148.5836 49.9515 90))
+    (property "Footprint" "Capacitor_SMD:C_0805_2012Metric_Pad1.18x1.45mm_HandSolder" (id 2) (at 148.59 52.705 0)
       (effects (font (size 1.27 1.27)) hide)
     )
@@
       (effects (font (size 1.27 1.27)) (justify left))
     )
-    (property "Footprint" "Resistor_SMD:R_2010_5025Metric" (id 2) (at 49.276 43.434 90)
+    (property "Footprint" "Resistor_SMD:R_0805_2012Metric_Pad1.20x1.40mm_HandSolder" (id 2) (at 49.276 43.434 90)
       (effects (font (size 1.27 1.27)) hide)
     )
@@
       (effects (font (size 1.27 1.27)) (justify left))
     )
-    (property "Footprint" "Resistor_SMD:R_2010_5025Metric" (id 2) (at 80.391 43.434 90)
+    (property "Footprint" "Resistor_SMD:R_0805_2012Metric_Pad1.20x1.40mm_HandSolder" (id 2) (at 80.391 43.434 90)
       (effects (font (size 1.27 1.27)) hide)
     )
@@
       (effects (font (size 1.27 1.27)) (justify left))
     )
-    (property "Footprint" "Resistor_SMD:R_2010_5025Metric" (id 2) (at 88.646 43.434 90)
+    (property "Footprint" "Resistor_SMD:R_0805_2012Metric_Pad1.20x1.40mm_HandSolder" (id 2) (at 88.646 43.434 90)
       (effects (font (size 1.27 1.27)) hide)
     )
@@
       (effects (font (size 1.27 1.27)) (justify left))
     )
-    (property "Footprint" "Resistor_SMD:R_2010_5025Metric_Pad1.40x2.65mm_HandSolder" (id 2) (at 198.501 56.134 90)
+    (property "Footprint" "Resistor_SMD:R_0805_2012Metric_Pad1.20x1.40mm_HandSolder" (id 2) (at 198.501 56.134 90)
       (effects (font (size 1.27 1.27)) hide)
     )
@@
       (effects (font (size 1.27 1.27)) (justify left))
     )
-    (property "Value" "0" (id 1) (at 199.136 41.8716 0)
-      (effects (font (size 1.27 1.27)) (justify left))
-    )
-    (property "Footprint" "Resistor_SMD:R_2010_5025Metric_Pad1.40x2.65mm_HandSolder" (id 2) (at 198.501 40.259 90)
+    (property "Value" "2k" (id 1) (at 199.136 41.8716 0)
+      (effects (font (size 1.27 1.27)) (justify left))
+    )
+    (property "Footprint" "Resistor_SMD:R_0805_2012Metric_Pad1.20x1.40mm_HandSolder" (id 2) (at 198.501 40.259 90)
       (effects (font (size 1.27 1.27)) hide)
     )
@@
       (effects (font (size 1.27 1.27)) (justify left))
     )
-    (property "Footprint" "Resistor_SMD:R_2010_5025Metric" (id 2) (at 32.131 43.434 90)
+    (property "Footprint" "Resistor_SMD:R_0805_2012Metric_Pad1.20x1.40mm_HandSolder" (id 2) (at 32.131 43.434 90)
       (effects (font (size 1.27 1.27)) hide)
     )
@@
       (effects (font (size 1.27 1.27)) (justify left))
     )
-    (property "Footprint" "Capacitor_SMD:C_1210_3225Metric_Pad1.33x2.70mm_HandSolder" (id 2) (at 197.485 66.675 0)
+    (property "Footprint" "Capacitor_SMD:C_0805_2012Metric_Pad1.18x1.45mm_HandSolder" (id 2) (at 197.485 66.675 0)
       (effects (font (size 1.27 1.27)) hide)
     )
@@
       (effects (font (size 1.27 1.27)) (justify left))
     )
-    (property "Footprint" "Resistor_SMD:R_2010_5025Metric" (id 2) (at 64.516 43.434 90)
+    (property "Footprint" "Resistor_SMD:R_0805_2012Metric_Pad1.20x1.40mm_HandSolder" (id 2) (at 64.516 43.434 90)
       (effects (font (size 1.27 1.27)) hide)
     )
@@
       (effects (font (size 1.27 1.27)) (justify left))
     )
-    (property "Footprint" "Resistor_SMD:R_2010_5025Metric" (id 2) (at 57.531 43.434 90)
+    (property "Footprint" "Resistor_SMD:R_0805_2012Metric_Pad1.20x1.40mm_HandSolder" (id 2) (at 57.531 43.434 90)
       (effects (font (size 1.27 1.27)) hide)
     )
@@
     (property "Reference" "C2" (id 0) (at 85.0836 102.4214 90))
     (property "Value" "10nf" (id 1) (at 85.0836 105.1965 90))
-    (property "Footprint" "Capacitor_SMD:C_1210_3225Metric_Pad1.33x2.70mm_HandSolder" (id 2) (at 85.09 107.95 0)
+    (property "Footprint" "Capacitor_SMD:C_0805_2012Metric_Pad1.18x1.45mm_HandSolder" (id 2) (at 85.09 107.95 0)
       (effects (font (size 1.27 1.27)) hide)
     )
@@
     )
     (path "/3871c7f7-59dd-41ed-b610-089a654b78c9"
-      (reference "C1") (unit 1) (value "0.1uf") (footprint "Capacitor_SMD:C_1210_3225Metric_Pad1.33x2.70mm_HandSolder")
+      (reference "C1") (unit 1) (value "0.01uf") (footprint "Capacitor_SMD:C_0805_2012Metric_Pad1.18x1.45mm_HandSolder")
     )
     (path "/e3fd266f-2205-4304-b250-0a7b5513e57e"
-      (reference "C2") (unit 1) (value "10nf") (footprint "Capacitor_SMD:C_1210_3225Metric_Pad1.33x2.70mm_HandSolder")
+      (reference "C2") (unit 1) (value "10nf") (footprint "Capacitor_SMD:C_0805_2012Metric_Pad1.18x1.45mm_HandSolder")
     )
     (path "/b322f59a-181e-4c1f-b178-c429a6fc4c9c"
-      (reference "C3") (unit 1) (value "22uf") (footprint "Capacitor_SMD:C_1210_3225Metric_Pad1.33x2.70mm_HandSolder")
+      (reference "C3") (unit 1) (value "22uf") (footprint "Capacitor_SMD:C_0805_2012Metric_Pad1.18x1.45mm_HandSolder")
     )
     (path "/cd1cff81-9d8a-4511-96d6-4ddb79484001"
@@
     )
     (path "/adabd5de-fc4a-417d-a1c8-2bbd07fdcae3"
-      (reference "R1") (unit 1) (value "100") (footprint "Resistor_SMD:R_2010_5025Metric")
+      (reference "R1") (unit 1) (value "100") (footprint "Resistor_SMD:R_0805_2012Metric_Pad1.20x1.40mm_HandSolder")
     )
     (path "/2cb24424-ef15-46ea-a53f-c332059a0409"
-      (reference "R2") (unit 1) (value "100") (footprint "Resistor_SMD:R_2010_5025Metric")
+      (reference "R2") (unit 1) (value "100") (footprint "Resistor_SMD:R_0805_2012Metric_Pad1.20x1.40mm_HandSolder")
     )
     (path "/3993c009-2498-46bd-a3f0-cf0d59d3f850"
-      (reference "R3") (unit 1) (value "100") (footprint "Resistor_SMD:R_2010_5025Metric")
+      (reference "R3") (unit 1) (value "100") (footprint "Resistor_SMD:R_0805_2012Metric_Pad1.20x1.40mm_HandSolder")
     )
     (path "/cff1fb99-003d-4be6-b312-75886921796e"
-      (reference "R4") (unit 1) (value "100") (footprint "Resistor_SMD:R_2010_5025Metric")
+      (reference "R4") (unit 1) (value "100") (footprint "Resistor_SMD:R_0805_2012Metric_Pad1.20x1.40mm_HandSolder")
     )
     (path "/c8251b44-bff7-440a-ba89-55eabc2e21f9"
-      (reference "R5") (unit 1) (value "100") (footprint "Resistor_SMD:R_2010_5025Metric")
+      (reference "R5") (unit 1) (value "100") (footprint "Resistor_SMD:R_0805_2012Metric_Pad1.20x1.40mm_HandSolder")
     )
     (path "/1072d4f3-8a89-4e33-a821-7fb9b181a953"
-      (reference "R6") (unit 1) (value "100") (footprint "Resistor_SMD:R_2010_5025Metric")
+      (reference "R6") (unit 1) (value "100") (footprint "Resistor_SMD:R_0805_2012Metric_Pad1.20x1.40mm_HandSolder")
     )
     (path "/44900aef-964f-46ab-bb2c-73b502ffeeed"
-      (reference "R7") (unit 1) (value "100") (footprint "Resistor_SMD:R_2010_5025Metric")
+      (reference "R7") (unit 1) (value "100") (footprint "Resistor_SMD:R_0805_2012Metric_Pad1.20x1.40mm_HandSolder")
     )
     (path "/45ca8d2b-1852-4185-9f1d-6f90169893f8"
-      (reference "R8") (unit 1) (value "100") (footprint "Resistor_SMD:R_2010_5025Metric")
+      (reference "R8") (unit 1) (value "100") (footprint "Resistor_SMD:R_0805_2012Metric_Pad1.20x1.40mm_HandSolder")
     )
     (path "/a0c05746-4db5-46c4-a2c6-7ac7750fd97a"
-      (reference "R9") (unit 1) (value "0") (footprint "Resistor_SMD:R_2010_5025Metric_Pad1.40x2.65mm_HandSolder")
+      (reference "R9") (unit 1) (value "2k") (footprint "Resistor_SMD:R_0805_2012Metric_Pad1.20x1.40mm_HandSolder")
     )
     (path "/51c415d5-32ed-4d26-b2fe-e2c8657ba45e"
-      (reference "R10") (unit 1) (value "13K") (footprint "Resistor_SMD:R_2010_5025Metric_Pad1.40x2.65mm_HandSolder")
+      (reference "R10") (unit 1) (value "13K") (footprint "Resistor_SMD:R_0805_2012Metric_Pad1.20x1.40mm_HandSolder")
     )
     (path "/b746016f-95c5-4b64-bbc8-f91857dc0514"

Commit message: Fixed the problem of the battery holder being the wrong way
Connections:
- net GND: now also BT1.1 (+); no longer BT1.2 (-)
- net VCC: now also BT1.2 (-); no longer BT1.1 (+)
Other:
- note added: "Reversed due to pin layout on the footprint"
Changed lines of the file:
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@@
+    (effects (font (size 1.27 1.27)) (justify left bottom))
+  )
+  (text "Reversed due to pin layout on the footprint\n" (at 103.124 26.924 0)
     (effects (font (size 1.27 1.27)) (justify left bottom))
   )
@@
     )
   )
-  (global_label "VCC" (shape input) (at 114.3 30.0056 0) (fields_autoplaced)
-    (effects (font (size 1.27 1.27)) (justify left))
-    (property "Intersheet References" "${INTERSHEET_REFS}" (id 0) (at 120.3417 29.9262 0)
-      (effects (font (size 1.27 1.27)) (justify left) hide)
-    )
-  )
   (global_label "LED_C" (shape input) (at 111.76 83.82 0) (fields_autoplaced)
     (effects (font (size 1.27 1.27)) (justify left))
@@
     (property "Intersheet References" "${INTERSHEET_REFS}" (id 0) (at 53.2606 114.8686 90)
       (effects (font (size 1.27 1.27)) (justify right) hide)
+    )
+  )
+  (global_label "GND" (shape input) (at 114.3 29.972 0) (fields_autoplaced)
+    (effects (font (size 1.27 1.27)) (justify left))
+    (property "Intersheet References" "${INTERSHEET_REFS}" (id 0) (at 120.5836 29.8926 0)
+      (effects (font (size 1.27 1.27)) (justify left) hide)
     )
   )
@@
     )
   )
+  (global_label "VCC" (shape input) (at 118.745 50.8 0) (fields_autoplaced)
+    (effects (font (size 1.27 1.27)) (justify left))
+    (property "Intersheet References" "${INTERSHEET_REFS}" (id 0) (at 124.7867 50.7206 0)
+      (effects (font (size 1.27 1.27)) (justify left) hide)
+    )
+  )
   (global_label "GND" (shape input) (at 167.005 70.485 270) (fields_autoplaced)
     (effects (font (size 1.27 1.27)) (justify right))
@@
     )
   )
-  (global_label "GND" (shape input) (at 118.745 50.8 0) (fields_autoplaced)
-    (effects (font (size 1.27 1.27)) (justify left))
-    (property "Intersheet References" "${INTERSHEET_REFS}" (id 0) (at 125.0286 50.7206 0)
-      (effects (font (size 1.27 1.27)) (justify left) hide)
-    )
-  )
